File: hardware/Voda septik.kicad_pcb (KiCad board)
At the start: 2 copper layers, 67.7 x 86.4 mm, 41 parts, among them J1 Napájení a 4-20mA senzory, J2 Screw_Terminal_01x09, J3 Display LCD I2C, J4 Display TM1637, U1 DC-DC 24V -> 5V, U2 MAX3485-modul, U3 ADS1115IDGS, U4 ESP32-DevKitC, U5 CA56-12CGKWA

Commit message: Dokreslit propojku RDY/ALERT
Parts:
- C2, C3, C4: value 100n -> 330n
Connections:
- net Net-(J2-A_RS485_elektroměr) renamed /RS485_A
- net Net-(J2-B_RS485_elektroměr) renamed /RS485_B
- net Net-(U3-AIN2) renamed /tlak_pred_filtrem
- U3 pad 6: unconnected-(U3-ALERT/RDY-Pad6) -> Net-(U3-ALERT/RDY)
- U4 pad 26: unconnected-(U4-ADC2_CH0/GPIO4-Pad26) -> Net-(U3-ALERT/RDY)
Routing:
- net Net-(U3-ALERT/RDY): track 0.00 -> 22.6 mm
